File: BPF.kicad_sch (KiCad schematic)
At the start: 2 parts, among them J2 IN-BPF

Commit message: Add files via upload
Added "WIP" branch, which is some of my mods.
Parts:
- renumbered BPF1 to J3
Changed lines of the file:
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@@
-(kicad_sch (version 20211123) (generator eeschema)
+(kicad_sch (version 20230121) (generator eeschema)
   (paper "A4")
   (wire (pts (xy 102.87 55.88) (xy 107.95 55.88))
-    (stroke (width 0) (type default) (color 0 0 0 0))
+    (stroke (width 0) (type default))
   )
   (wire (pts (xy 154.94 55.88) (xy 148.59 55.88))
-    (stroke (width 0) (type default) (color 0 0 0 0))
+    (stroke (width 0) (type default))
   )
-  (hierarchical_label "BPF-OUT" (shape output) (at 154.94 55.88 0)
+  (hierarchical_label "BPF-OUT" (shape output) (at 154.94 55.88 0) (fields_autoplaced)
     (effects (font (size 1.27 1.27)) (justify left))
   )
-  (hierarchical_label "BPF-IN" (shape input) (at 102.87 55.88 180)
+  (hierarchical_label "BPF-IN" (shape input) (at 102.87 55.88 180) (fields_autoplaced)
     (effects (font (size 1.27 1.27)) (justify right))
   )
   (symbol (lib_id "Connector:Conn_01x03_Female") (at 113.03 55.88 0) (unit 1)
-    (in_bom yes) (on_board yes)
-    (property "Reference" "J2" (id 0) (at 110.49 48.26 0)
+    (in_bom yes) (on_board yes) (dnp no)
+    (property "Reference" "J2" (at 110.49 48.26 0)
       (effects (font (size 1.27 1.27)) (justify left))
     )
-    (property "Value" "IN-BPF" (id 1) (at 102.87 50.8 0)
+    (property "Value" "IN-BPF" (at 102.87 50.8 0)
       (effects (font (size 1.27 1.27)) (justify left))
     )
-    (property "Footprint" "Connector_PinSocket_2.54mm:PinSocket_1x03_P2.54mm_Vertical" (id 2) (at 113.03 55.88 0)
+    (property "Footprint" "Connector_PinSocket_2.54mm:PinSocket_1x03_P2.54mm_Vertical" (at 113.03 55.88 0)
       (effects (font (size 1.27 1.27)) hide)
     )
-    (property "Datasheet" "~" (id 3) (at 113.03 55.88 0)
+    (property "Datasheet" "~" (at 113.03 55.88 0)
       (effects (font (size 1.27 1.27)) hide)
     )
@@
     (pin "2")
     (pin "3")
+    (instances
+      (project "SDR-Transceiver"
+        (path "/09eb8c56-3cf8-43d0-96ec-95e0f12e2183/4b1ef805-7fd0-4a4a-b5da-5feeaa035c65"
+          (reference "J2") (unit 1)
+        )
+      )
+    )
   )
   (symbol (lib_id "power:GND") (at 107.95 53.34 0) (unit 1)
-    (in_bom yes) (on_board yes) (fields_autoplaced)
-    (property "Reference" "#PWR0152" (id 0) (at 107.95 59.69 0)
+    (in_bom yes) (on_board yes) (dnp no) (fields_autoplaced)
+    (property "Reference" "#PWR0152" (at 107.95 59.69 0)
       (effects (font (size 1.27 1.27)) hide)
     )
-    (property "Value" "GND" (id 1) (at 107.95 58.42 0))
-    (property "Footprint" "" (id 2) (at 107.95 53.34 0)
+    (property "Value" "GND" (at 107.95 58.42 0)
+      (effects (font (size 1.27 1.27)))
+    )
+    (property "Footprint" "" (at 107.95 53.34 0)
       (effects (font (size 1.27 1.27)) hide)
     )
-    (property "Datasheet" "" (id 3) (at 107.95 53.34 0)
+    (property "Datasheet" "" (at 107.95 53.34 0)
       (effects (font (size 1.27 1.27)) hide)
     )
     (pin "1")
+    (instances
+      (project "SDR-Transceiver"
+        (path "/09eb8c56-3cf8-43d0-96ec-95e0f12e2183/4b1ef805-7fd0-4a4a-b5da-5feeaa035c65"
+          (reference "#PWR0152") (unit 1)
+        )
+      )
+    )
   )
   (symbol (lib_id "Connector:Conn_01x03_Female") (at 143.51 55.88 0) (mirror y) (unit 1)
-    (in_bom yes) (on_board yes) (fields_autoplaced)
-    (property "Reference" "BPF1" (id 0) (at 144.145 48.26 0))
-    (property "Value" "OUT-BPF" (id 1) (at 144.145 50.8 0))
-    (property "Footprint" "Connector_PinSocket_2.54mm:PinSocket_1x03_P2.54mm_Vertical" (id 2) (at 143.51 55.88 0)
+    (in_bom yes) (on_board yes) (dnp no) (fields_autoplaced)
+    (property "Reference" "J3" (at 144.145 48.26 0)
+      (effects (font (size 1.27 1.27)))
+    )
+    (property "Value" "OUT-BPF" (at 144.145 50.8 0)
+      (effects (font (size 1.27 1.27)))
+    )
+    (property "Footprint" "Connector_PinSocket_2.54mm:PinSocket_1x03_P2.54mm_Vertical" (at 143.51 55.88 0)
       (effects (font (size 1.27 1.27)) hide)
     )
-    (property "Datasheet" "~" (id 3) (at 143.51 55.88 0)
+    (property "Datasheet" "~" (at 143.51 55.88 0)
       (effects (font (size 1.27 1.27)) hide)
     )
@@
     (pin "2")
     (pin "3")
+    (instances
+      (project "SDR-Transceiver"
+        (path "/09eb8c56-3cf8-43d0-96ec-95e0f12e2183/4b1ef805-7fd0-4a4a-b5da-5feeaa035c65"
+          (reference "J3") (unit 1)
+        )
+      )
+    )
   )
   (symbol (lib_id "power:GND") (at 148.59 58.42 0) (unit 1)
-    (in_bom yes) (on_board yes) (fields_autoplaced)
-    (property "Reference" "#PWR0103" (id 0) (at 148.59 64.77 0)
+    (in_bom yes) (on_board yes) (dnp no) (fields_autoplaced)
+    (property "Reference" "#PWR0103" (at 148.59 64.77 0)
       (effects (font (size 1.27 1.27)) hide)
     )
-    (property "Value" "GND" (id 1) (at 148.59 63.5 0))
-    (property "Footprint" "" (id 2) (at 148.59 58.42 0)
+    (property "Value" "GND" (at 148.59 63.5 0)
+      (effects (font (size 1.27 1.27)))
+    )
+    (property "Footprint" "" (at 148.59 58.42 0)
       (effects (font (size 1.27 1.27)) hide)
     )
-    (property "Datasheet" "" (id 3) (at 148.59 58.42 0)
+    (property "Datasheet" "" (at 148.59 58.42 0)
       (effects (font (size 1.27 1.27)) hide)
     )
     (pin "1")
+    (instances
+      (project "SDR-Transceiver"
+        (path "/09eb8c56-3cf8-43d0-96ec-95e0f12e2183/4b1ef805-7fd0-4a4a-b5da-5feeaa035c65"
+          (reference "#PWR0103") (unit 1)
+        )
+      )
+    )
   )
   (symbol (lib_id "power:GND") (at 148.59 53.34 0) (unit 1)
-    (in_bom yes) (on_board yes) (fields_autoplaced)
-    (property "Reference" "#PWR0153" (id 0) (at 148.59 59.69 0)
+    (in_bom yes) (on_board yes) (dnp no) (fields_autoplaced)
+    (property "Reference" "#PWR0153" (at 148.59 59.69 0)
       (effects (font (size 1.27 1.27)) hide)
     )
-    (property "Value" "GND" (id 1) (at 148.59 58.42 0))
-    (property "Footprint" "" (id 2) (at 148.59 53.34 0)
+    (property "Value" "GND" (at 148.59 58.42 0)
+      (effects (font (size 1.27 1.27)))
+    )
+    (property "Footprint" "" (at 148.59 53.34 0)
       (effects (font (size 1.27 1.27)) hide)
     )
-    (property "Datasheet" "" (id 3) (at 148.59 53.34 0)
+    (property "Datasheet" "" (at 148.59 53.34 0)
       (effects (font (size 1.27 1.27)) hide)
     )
     (pin "1")
+    (instances
+      (project "SDR-Transceiver"
+        (path "/09eb8c56-3cf8-43d0-96ec-95e0f12e2183/4b1ef805-7fd0-4a4a-b5da-5feeaa035c65"
+          (reference "#PWR0153") (unit 1)
+        )
+      )
+    )
   )
   (symbol (lib_id "power:GND") (at 107.95 58.42 0) (unit 1)
-    (in_bom yes) (on_board yes) (fields_autoplaced)
-    (property "Reference" "#PWR0102" (id 0) (at 107.95 64.77 0)
+    (in_bom yes) (on_board yes) (dnp no) (fields_autoplaced)
+    (property "Reference" "#PWR0102" (at 107.95 64.77 0)
       (effects (font (size 1.27 1.27)) hide)
     )
-    (property "Value" "GND" (id 1) (at 107.95 63.5 0))
-    (property "Footprint" "" (id 2) (at 107.95 58.42 0)
+    (property "Value" "GND" (at 107.95 63.5 0)
+      (effects (font (size 1.27 1.27)))
+    )
+    (property "Footprint" "" (at 107.95 58.42 0)
       (effects (font (size 1.27 1.27)) hide)
     )
-    (property "Datasheet" "" (id 3) (at 107.95 58.42 0)
+    (property "Datasheet" "" (at 107.95 58.42 0)
       (effects (font (size 1.27 1.27)) hide)
     )
     (pin "1")
+    (instances
+      (project "SDR-Transceiver"
+        (path "/09eb8c56-3cf8-43d0-96ec-95e0f12e2183/4b1ef805-7fd0-4a4a-b5da-5feeaa035c65"
+          (reference "#PWR0102") (unit 1)
+        )
+      )
+    )
   )
 )
