File: DSP.kicad_sch (KiCad schematic)
At the start: 24 parts, among them J10 USB to Serial, J11 LCD, Q4 2N3904-SMD, Q5 2N3904-SMD, Q6 AO3400A, SW1 RST, SW2 Frequency, SW3 Menu, SW4 BOOT, U6 ESP32-A1S

Commit message: Add files via upload
Added "WIP" branch, which is some of my mods.
Parts:
- removed C24, C26: 22uF, Capacitor_SMD:CP_Elec_4x4.5, symbol Device:C_Polarized
- removed C25, C27, C50, C51: 1uF, Capacitor_SMD:C_1206_3216Metric, symbol Xenir:Capacitor
- removed C28, C29: .1uF, Capacitor_SMD:C_1206_3216Metric, symbol Xenir:Capacitor
- removed J10: USB to Serial, Connector_PinSocket_2.54mm:PinSocket_1x07_P2.54mm_Vertical, symbol Connector:Conn_01x07_Female
- removed J11: LCD, Connector_PinSocket_2.54mm:PinSocket_1x04_P2.54mm_Vertical, symbol Connector_Generic:Conn_01x04
- removed Q4, Q5: 2N3904-SMD, Package_TO_SOT_SMD:SOT-23, symbol Tayloe-Mixer-v3-rescue:2N3904-SMD-xenir
- removed Q6: AO3400A, Package_TO_SOT_SMD:SOT-23, symbol Transistor_FET:AO3400A
- removed R21, R22: 330, Resistor_SMD:R_0805_2012Metric, symbol Xenir:Resistor
- removed R44, R45: 10k, Resistor_SMD:R_0805_2012Metric, symbol Tayloe-Mixer-v3-rescue:Resistor-Xenir-esp32-a1s-rescue
- removed R46: 1k, Resistor_SMD:R_0805_2012Metric, symbol xenir:Resistor
- removed R47: 10k, Resistor_SMD:R_0805_2012Metric, symbol xenir:Resistor
- removed SW1: RST, Button_Switch_SMD:SW_SPST_B3U-1000P, symbol Switch:SW_DIP_x01
- removed SW4: BOOT, Button_Switch_SMD:SW_SPST_B3U-1000P, symbol Switch:SW_DIP_x01
- removed U6: ESP32-A1S, xenir_v6:esp32-a1s-header, symbol Xenir:ESP32-A1S
- added C59, C61, C62, C65, C66, C67, C68, C69, C70, C71: 100nF, Capacitor_SMD:C_0402_1005Metric, symbol Device:C_Small
- added C60, C64: 1uF, Capacitor_SMD:C_0402_1005Metric, symbol Device:C_Small
- added C63: 10uF, Capacitor_SMD:C_0402_1005Metric, symbol Device:C_Small
- added D3: HEARTBEAT, symbol Device:LED_Small
- added D4: PWR_ON, symbol Device:LED_Small
- added F1: 500mA, Fuse:Fuse_1206_3216Metric, symbol Device:Polyfuse_Small
- added J14: USBC, Connector_USB:USB_C_Receptacle_HRO_TYPE-C-31-M-12, symbol Connector:USB_C_Receptacle_USB2.0
- added J9: SWD, Connector_PinSocket_2.54mm:PinSocket_1x05_P2.54mm_Vertical, symbol Connector_Generic:Conn_01x05
- added R21, R22: 1K5, Resistor_SMD:R_0402_1005Metric, symbol Device:R_Small
- added R25, R30: 1k, Resistor_SMD:R_0402_1005Metric, symbol Device:R_Small
- added R26, R27: 27R, Resistor_SMD:R_0603_1608Metric, symbol Device:R_Small
- added R28, R29: 5k1, Resistor_SMD:R_0402_1005Metric, symbol Device:R_Small
- added R43: 10k, Resistor_SMD:R_0402_1005Metric, symbol Device:R_Small
- added SW1: USR, Connector_PinSocket_2.54mm:PinSocket_1x02_P2.54mm_Vertical, symbol Switch:SW_Push
- added SW4: Reset, Connector_PinSocket_2.54mm:PinSocket_1x02_P2.54mm_Vertical, symbol Switch:SW_Push
- added SW5: SW_Push, Connector_PinSocket_2.54mm:PinSocket_1x02_P2.54mm_Vertical, symbol Switch:SW_Push
- added U14: W25Q128JVS, Package_SO:SOIC-8_5.23x5.23mm_P1.27mm, symbol Memory_Flash:W25Q128JVS
- added U15: USBLC6-2SC6, Package_TO_SOT_SMD:SOT-23-6, symbol Power_Protection:USBLC6-2SC6
- added U6: RP2040, Sleep-Lib:RP2040-QFN-56, symbol Sleep-lib:RP2040
Connections:
- net +3V3: now also C59.1, C63.1, C64.1, C65.1, C66.1, C67.1, C68.1, C69.1, C70.1, C71.1, J9.2 (Pin_2), R22.2, R25.1, R43.1, U14.8 (VCC), U6.1 (IOVDD), U6.10 (IOVDD), U6.22 (IOVDD), U6.33 (IOVDD), U6.42 (IOVDD), U6.43 (ADC_AVDD), U6.44 (VREG_VIN), U6.48 (USB_VDD), U6.49 (IOVDD)
- net +5V: now also F1.2
- net GND: now also C59.2, C60.2, C61.2, C62.2, C63.2, C64.2, C65.2, C66.2, C67.2, C68.2, C69.2, C70.2, C71.2, D3.1 (K), D4.1 (K), J14.A1 (GND), J14.A12 (GND), J14.B1 (GND), J14.B12 (GND), J14.S1 (SHIELD), J9.3 (Pin_3), R28.2, R29.2, SW1.1, SW4.1, SW5.1, U14.4 (GND), U15.2 (GND), U6.19 (TESTEN), U6.57 (GND); no longer SW2.C
- net GPIO13: now also U6.16 (GPIO13)
- net GPIO14: now also U6.17 (GPIO14)
- net GPIO15: now also U6.18 (GPIO15)
- net GPIO4: now also U6.6 (GPIO4)
- net GPIO12: no longer names the net of SW2.S2
- net GPIO2 renamed GPIO34
- new net: D4.2 (A), R22.1
- new net: D3.2 (A), R21.1
- new net: U14.2 (DO(IO1)), U6.55 (QSPI_SD1)
- new net: U14.3 (IO2), U6.54 (QSPI_SD2)
- new net: U14.5 (DI(IO0)), U6.53 (QSPI_SD0)
- new net: U14.7 (IO3), U6.51 (QSPI_SD3)
- new net +1V1: C60.1, C61.1, C62.1, U6.23 (DVDD), U6.45 (VREG_VOUT), U6.50 (DVDD)
- new net BOOT: R30.1, SW5.2
- new net CC1: J14.A5 (CC1), R28.1
- new net CC2: J14.B5 (CC2), R29.1
- new net CS: R30.2, U14.1 (~{CS}), U6.56 (QSPI_SS_N)
- new net DDS_DRCTL: U6.38 (GPIO26/ADC0)
- new net DDS_EXT_PWR_DWN: U6.35 (GPIO23)
- new net DDS_IO_RST: U6.30 (GPIO19)
- new net DDS_IO_UPDATE: U6.32 (GPIO21)
- new net DDS_MR_REST: U6.34 (GPIO22)
- new net DDS_OSK: U6.31 (GPIO20)
- new net DDS_P0: U6.39 (GPIO27/ADC1)
- new net DDS_P1: U6.40 (GPIO28/ADC2)
- new net DDS_P2: U6.41 (GPIO29/ADC3)
- new net D_+: R26.2, U6.47 (D+)
- new net D_-: R27.2, U6.46 (D-)
- new net D_N: R27.1, U15.3 (I/O2)
- new net D_P: R26.1, U15.1 (I/O1)
- new net D_USB_N: J14.A7 (D-), J14.B7 (D-), U15.4 (I/O2)
- new net D_USB_P: J14.A6 (D+), J14.B6 (D+), U15.6 (I/O1)
- new net GPIO24: R43.2, SW1.2, U6.36 (GPIO24)
- new net GPIO25: R21.2, U6.37 (GPIO25)
- new net I2C0_SCL: U6.7 (GPIO5)
- new net I2C1_SCL: U6.9 (GPIO7)
- new net I2C1_SDA: U6.8 (GPIO6)
- new net PIO0_I2S0_OUT: U6.15 (GPIO12)
- new net QSPI_CLK: U14.6 (CLK), U6.52 (QSPI_SCLK)
- new net SPI0_CSN: U6.3 (GPIO1)
- new net SPI0_MISO: U6.2 (GPIO0)
- new net SPI0_MOSI: U6.5 (GPIO3)
- new net SPI0_SCK: U6.4 (GPIO2)
- new net SPI1_CSN: U6.12 (GPIO9)
- new net SPI1_MISO: U6.11 (GPIO8)
- new net SPI1_MOSI: U6.14 (GPIO11)
- new net SPI1_SCK: U6.13 (GPIO10)
- new net SWCLK: J9.5 (Pin_5), U6.24 (SWCLK)
- new net SWD: J9.4 (Pin_4), U6.25 (SWDIO)
- new net TFT_BLK: U6.29 (GPIO18)
- new net TFT_DC: U6.28 (GPIO17)
- new net TFT_RES: U6.27 (GPIO16)
- new net VBUS: F1.1, J14.A4 (VBUS), J14.A9 (VBUS), J14.B4 (VBUS), J14.B9 (VBUS)
- new net XTAL_IN: U6.20 (XTAL_IN)
- new net XTAL_OUT: U6.21 (XTAL_OUT)
- new net ~{RESET}: J9.1 (Pin_1), R25.2, U6.26 (~{RUN})
- no-connect marks 0 -> 2
Other:
- note added: "DDS_CS"
- moved on the sheet: SW2, SW3
