File: LPF.kicad_sch (KiCad schematic)
At the start: 2 parts, among them J4 IN-LPF

Commit message: Add files via upload
Added "WIP" branch, which is some of my mods.
Parts:
- renumbered LPF1 to J5
Changed lines of the file:
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@@
-(kicad_sch (version 20211123) (generator eeschema)
+(kicad_sch (version 20230121) (generator eeschema)
   (paper "A4")
   (wire (pts (xy 105.41 83.82) (xy 110.49 83.82))
-    (stroke (width 0) (type default) (color 0 0 0 0))
+    (stroke (width 0) (type default))
   )
   (wire (pts (xy 157.48 83.82) (xy 151.13 83.82))
-    (stroke (width 0) (type default) (color 0 0 0 0))
+    (stroke (width 0) (type default))
   )
-  (hierarchical_label "OUT-LPF" (shape output) (at 157.48 83.82 0)
+  (hierarchical_label "OUT-LPF" (shape output) (at 157.48 83.82 0) (fields_autoplaced)
     (effects (font (size 1.27 1.27)) (justify left))
   )
-  (hierarchical_label "IN-LPF" (shape input) (at 105.41 83.82 180)
+  (hierarchical_label "IN-LPF" (shape input) (at 105.41 83.82 180) (fields_autoplaced)
     (effects (font (size 1.27 1.27)) (justify right))
   )
   (symbol (lib_id "power:GND") (at 110.49 86.36 0) (unit 1)
-    (in_bom yes) (on_board yes) (fields_autoplaced)
-    (property "Reference" "#PWR0101" (id 0) (at 110.49 92.71 0)
+    (in_bom yes) (on_board yes) (dnp no) (fields_autoplaced)
+    (property "Reference" "#PWR0101" (at 110.49 92.71 0)
       (effects (font (size 1.27 1.27)) hide)
     )
-    (property "Value" "GND" (id 1) (at 110.49 91.44 0))
-    (property "Footprint" "" (id 2) (at 110.49 86.36 0)
+    (property "Value" "GND" (at 110.49 91.44 0)
+      (effects (font (size 1.27 1.27)))
+    )
+    (property "Footprint" "" (at 110.49 86.36 0)
       (effects (font (size 1.27 1.27)) hide)
     )
-    (property "Datasheet" "" (id 3) (at 110.49 86.36 0)
+    (property "Datasheet" "" (at 110.49 86.36 0)
       (effects (font (size 1.27 1.27)) hide)
     )
     (pin "1")
+    (instances
+      (project "SDR-Transceiver"
+        (path "/09eb8c56-3cf8-43d0-96ec-95e0f12e2183/3c85d954-82ab-4b0c-952d-ee98ece6c954"
+          (reference "#PWR0101") (unit 1)
+        )
+      )
+    )
   )
   (symbol (lib_id "power:GND") (at 151.13 81.28 0) (unit 1)
-    (in_bom yes) (on_board yes) (fields_autoplaced)
-    (property "Reference" "#PWR0156" (id 0) (at 151.13 87.63 0)
+    (in_bom yes) (on_board yes) (dnp no) (fields_autoplaced)
+    (property "Reference" "#PWR0156" (at 151.13 87.63 0)
       (effects (font (size 1.27 1.27)) hide)
     )
-    (property "Value" "GND" (id 1) (at 151.13 86.36 0))
-    (property "Footprint" "" (id 2) (at 151.13 81.28 0)
+    (property "Value" "GND" (at 151.13 86.36 0)
+      (effects (font (size 1.27 1.27)))
+    )
+    (property "Footprint" "" (at 151.13 81.28 0)
       (effects (font (size 1.27 1.27)) hide)
     )
-    (property "Datasheet" "" (id 3) (at 151.13 81.28 0)
+    (property "Datasheet" "" (at 151.13 81.28 0)
       (effects (font (size 1.27 1.27)) hide)
     )
     (pin "1")
+    (instances
+      (project "SDR-Transceiver"
+        (path "/09eb8c56-3cf8-43d0-96ec-95e0f12e2183/3c85d954-82ab-4b0c-952d-ee98ece6c954"
+          (reference "#PWR0156") (unit 1)
+        )
+      )
+    )
   )
   (symbol (lib_id "power:GND") (at 110.49 81.28 0) (unit 1)
-    (in_bom yes) (on_board yes) (fields_autoplaced)
-    (property "Reference" "#PWR0154" (id 0) (at 110.49 87.63 0)
+    (in_bom yes) (on_board yes) (dnp no) (fields_autoplaced)
+    (property "Reference" "#PWR0154" (at 110.49 87.63 0)
       (effects (font (size 1.27 1.27)) hide)
     )
-    (property "Value" "GND" (id 1) (at 110.49 86.36 0))
-    (property "Footprint" "" (id 2) (at 110.49 81.28 0)
+    (property "Value" "GND" (at 110.49 86.36 0)
+      (effects (font (size 1.27 1.27)))
+    )
+    (property "Footprint" "" (at 110.49 81.28 0)
       (effects (font (size 1.27 1.27)) hide)
     )
-    (property "Datasheet" "" (id 3) (at 110.49 81.28 0)
+    (property "Datasheet" "" (at 110.49 81.28 0)
       (effects (font (size 1.27 1.27)) hide)
     )
     (pin "1")
+    (instances
+      (project "SDR-Transceiver"
+        (path "/09eb8c56-3cf8-43d0-96ec-95e0f12e2183/3c85d954-82ab-4b0c-952d-ee98ece6c954"
+          (reference "#PWR0154") (unit 1)
+        )
+      )
+    )
   )
   (symbol (lib_id "Connector:Conn_01x03_Female") (at 146.05 83.82 0) (mirror y) (unit 1)
-    (in_bom yes) (on_board yes) (fields_autoplaced)
-    (property "Reference" "LPF1" (id 0) (at 146.685 76.2 0))
-    (property "Value" "OUT-LPF" (id 1) (at 146.685 78.74 0))
-    (property "Footprint" "Connector_PinSocket_2.54mm:PinSocket_1x03_P2.54mm_Vertical" (id 2) (at 146.05 83.82 0)
+    (in_bom yes) (on_board yes) (dnp no) (fields_autoplaced)
+    (property "Reference" "J5" (at 146.685 76.2 0)
+      (effects (font (size 1.27 1.27)))
+    )
+    (property "Value" "OUT-LPF" (at 146.685 78.74 0)
+      (effects (font (size 1.27 1.27)))
+    )
+    (property "Footprint" "Connector_PinSocket_2.54mm:PinSocket_1x03_P2.54mm_Vertical" (at 146.05 83.82 0)
       (effects (font (size 1.27 1.27)) hide)
     )
-    (property "Datasheet" "~" (id 3) (at 146.05 83.82 0)
+    (property "Datasheet" "~" (at 146.05 83.82 0)
       (effects (font (size 1.27 1.27)) hide)
     )
@@
     (pin "2")
     (pin "3")
+    (instances
+      (project "SDR-Transceiver"
+        (path "/09eb8c56-3cf8-43d0-96ec-95e0f12e2183/3c85d954-82ab-4b0c-952d-ee98ece6c954"
+          (reference "J5") (unit 1)
+        )
+      )
+    )
   )
   (symbol (lib_id "Connector:Conn_01x03_Female") (at 115.57 83.82 0) (unit 1)
-    (in_bom yes) (on_board yes)
-    (property "Reference" "J4" (id 0) (at 113.03 76.2 0)
+    (in_bom yes) (on_board yes) (dnp no)
+    (property "Reference" "J4" (at 113.03 76.2 0)
       (effects (font (size 1.27 1.27)) (justify left))
     )
-    (property "Value" "IN-LPF" (id 1) (at 105.41 78.74 0)
+    (property "Value" "IN-LPF" (at 105.41 78.74 0)
       (effects (font (size 1.27 1.27)) (justify left))
     )
-    (property "Footprint" "Connector_PinSocket_2.54mm:PinSocket_1x03_P2.54mm_Vertical" (id 2) (at 115.57 83.82 0)
+    (property "Footprint" "Connector_PinSocket_2.54mm:PinSocket_1x03_P2.54mm_Vertical" (at 115.57 83.82 0)
       (effects (font (size 1.27 1.27)) hide)
     )
-    (property "Datasheet" "~" (id 3) (at 115.57 83.82 0)
+    (property "Datasheet" "~" (at 115.57 83.82 0)
       (effects (font (size 1.27 1.27)) hide)
     )
@@
     (pin "2")
     (pin "3")
+    (instances
+      (project "SDR-Transceiver"
+        (path "/09eb8c56-3cf8-43d0-96ec-95e0f12e2183/3c85d954-82ab-4b0c-952d-ee98ece6c954"
+          (reference "J4") (unit 1)
+        )
+      )
+    )
   )
   (symbol (lib_id "power:GND") (at 151.13 86.36 0) (unit 1)
-    (in_bom yes) (on_board yes) (fields_autoplaced)
-    (property "Reference" "#PWR0155" (id 0) (at 151.13 92.71 0)
+    (in_bom yes) (on_board yes) (dnp no) (fields_autoplaced)
+    (property "Reference" "#PWR0155" (at 151.13 92.71 0)
       (effects (font (size 1.27 1.27)) hide)
     )
-    (property "Value" "GND" (id 1) (at 151.13 91.44 0))
-    (property "Footprint" "" (id 2) (at 151.13 86.36 0)
+    (property "Value" "GND" (at 151.13 91.44 0)
+      (effects (font (size 1.27 1.27)))
+    )
+    (property "Footprint" "" (at 151.13 86.36 0)
       (effects (font (size 1.27 1.27)) hide)
     )
-    (property "Datasheet" "" (id 3) (at 151.13 86.36 0)
+    (property "Datasheet" "" (at 151.13 86.36 0)
       (effects (font (size 1.27 1.27)) hide)
     )
     (pin "1")
+    (instances
+      (project "SDR-Transceiver"
+        (path "/09eb8c56-3cf8-43d0-96ec-95e0f12e2183/3c85d954-82ab-4b0c-952d-ee98ece6c954"
+          (reference "#PWR0155") (unit 1)
+        )
+      )
+    )
   )
 )
