File: SDR-Transceiver.kicad_pcb (KiCad board)
At the start: 2 copper layers, 150 x 100 mm, 160 parts, among them J1 BNC, J10 USB to Serial, J11 LCD, J12 MIC, J13 Audio Out, J2 IN-BPF, J4 IN-LPF, J6 TO-PA, J7 FROM-PA, J8 Amplifier T/R, J9 Barrel_Jack_Switch, K1 G6S-2, K2 G6S-2, Q1 AO3400A, Q2 AO3400A, Q3 2N2222, Q4 2N3904-SMD, Q5 2N3904-SMD, Q6 AO3400A, SW1 RST, SW2 Frequency, SW3 Menu, SW4 BOOT, T3 T50_SPLITTER, T4 T50_COMBINER, U1 FST3253, U10 si5351, U11 LM358, U2 LM4562, U3 FST3253, U4 LM4562, U5 LM4562, U6 ESP32-A1S, U7 FST3257, U8 L7805, U9 AMS1117CD-3.3

Commit message: Add files via upload
Added "WIP" branch, which is some of my mods.
Parts:
- removed C56, C57, C58: .1uF, Capacitor_SMD:C_1206_3216Metric
- C28, C29: value .1uF -> 1uF
- renumbered BPF1 to J3, LPF1 to J5
Connections:
- SW3 pad A: GPIO2 -> GPIO34
- U6 pad 11: GPIO2 -> unconnected-(U6-Pad11)
- U6 pad 5: unconnected-(U6-Pad5) -> GPIO34
Routing:
- net GPIO34: track 0.00 -> 71.6 mm, vias 0 -> 1
- net GPIO2: track 55.5 -> 0.00 mm
- net Encoder2.5: track 55.6 -> 50.5 mm
- net Net-(C49-Pad1): track 30.5 -> 27.1 mm
Other:
- board text removed: "Amplifier T/R"
- board text removed: "Antenna"
- board text removed: "Audio Out"
- board text removed: "Audio Switch"
- board text removed: "BPF"
- board text removed: "From PA"
- board text removed: "LO"
- board text removed: "LPF"
- board text removed: "Mic Preamp"
- board text removed: "Microphone"
- board text removed: "NA5Y"
- board text removed: "Power"
- board text removed: "RF Switch"
- board text removed: "SDR Transceiver"
- board text removed: "Tayloe Decoder"
- board text removed: "Tayloe Encoder"
- board text removed: "To PA"
