File: SDR-Transceiver.kicad_sch (KiCad schematic)
At the start: 5 parts, among them J1 BNC

Commit message: Add files via upload
Added "WIP" branch, which is some of my mods.
Connections:
- no-connect marks 0 -> 2
Other:
- sheet Audio Switch renamed Audio Interface
- sheet Audio Interface ports: added AUX, Analog_en, CAD/CSN, DeMod_I, DeMod_Q, EarPhone, Enc_I, Enc_Q, I2S0, I2S1, I2S1_O, I2S2_O, MISO/SDA, MOSI, Mic, SCK/SCL, SCL, SDA, SPK; removed INL, INL1, INL2, INR, INR1, INR2, OUTL, OUTL1, OUTL2, OUTR, OUTR1, OUTR2
- note added: "I2S Transmit and Receive BUSs"
- note added: "IQ Demod Path"
- note added: "IQ Mod Path"
