File: mic.kicad_sch (KiCad schematic)
At the start: 11 parts, among them J12 MIC, U11 LM358

Commit message: Add files via upload
Added "WIP" branch, which is some of my mods.
Parts:
- removed R52: 5.1k, Resistor_SMD:R_0805_2012Metric, symbol mic-preamp-rescue:Resistor-Xenir
- removed R53, R54: 10k, Resistor_SMD:R_0805_2012Metric, symbol mic-preamp-rescue:Resistor-Xenir
- removed R55: 1k, Resistor_SMD:R_0805_2012Metric, symbol mic-preamp-rescue:Resistor-Xenir
- removed R56: 100k, Resistor_SMD:R_0805_2012Metric, symbol mic-preamp-rescue:Resistor-Xenir
- added R24 (x5): 2K2, Resistor_SMD:R_0805_2012Metric_Pad1.20x1.40mm_HandSolder, symbol Device:R
- U11: footprint xenir:SOIC8 -> Package_SO:SO-5_4.4x3.6mm_P1.27mm
Connections:
- net +5V: now also R24.1, R24.1
- net GND: now also R24.2
- net MICIN: now also R24.2
- net at U11.5 (+IN): now also R24.1, R24.2
- net at C52.2: now also R24.1
- net at C54.2, U11.6 (-IN): now also R24.1, R24.2
- net at C54.1, C55.2, U11.7 (OUT): now also R24.2
