File: taylor-detector.kicad_sch (KiCad schematic)
At the start: 18 parts, among them T3 T50_SPLITTER, U1 FST3253, U2 LM4562

Commit message: Add files via upload
Added "WIP" branch, which is some of my mods.
Parts:
- removed C56: .1uF, Capacitor_SMD:C_1206_3216Metric, symbol Xenir:Capacitor
- removed T3: T50_SPLITTER, Xenir:T50 Trifilar, symbol Xenir:T50_SPLITTER
- added C?: C_value?, Capacitor_SMD:C_0805_2012Metric_Pad1.18x1.45mm_HandSolder, symbol Device:C
- added R? (x2): 0R, Resistor_SMD:R_0805_2012Metric_Pad1.20x1.40mm_HandSolder, symbol Device:R
- added TR?: TC1-1T+, RF_Mini-Circuits:Mini-Circuits_CD637_H5.23mm, symbol Transformer:ADT1-6T
- added U? (x2): LT6231, Xenir:SO08, symbol Amplifier_Operational:LM358
- C11, C12, C13, C14: value 470nF -> 220nF
- C15, C16: value 1nF -> NC
- R1, R2, R3, R4: value 100 -> 0R
- U2: value LM4562 -> LT6231
Connections:
- net Detector-180 is gone; now on net Detector-0: C13.2, R3.1, U1.13 (2B4), U1.6 (1B1)
- net Detector-270 is gone; now on net Detector-0: C14.2, R4.1, U1.12 (2B3), U1.5 (1B2)
- net Detector-90 is gone; now on net Detector-0: C12.2, R2.1, U1.11 (2B2), U1.4 (1B3)
- net +2V5: now also TR?.5
- net Detector-In: now also C?.1, TR?.3
- net GND: now also C?.2, TR?.1
- net at U1.7 (1A): now also R?.2
- net at U1.9 (2A): now also R?.2
- new net: R?.1, TR?.4
- new net: R?.1, TR?.6
Other:
- note added: "This has a tuned input at 8Mhz. This is an IF frequency As this is a single conversion receiver and transmitter running an 8mHz immediate frequency."
- moved on the sheet: C10, C11, C12, C13, C14, C15, C16, C9, R1, R2, R3, R4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
