File: taylor-encoder.kicad_sch (KiCad schematic)
At the start: 37 parts, among them T4 T50_COMBINER, U3 FST3253, U4 LM4562, U5 LM4562

Commit message: Add files via upload
Added "WIP" branch, which is some of my mods.
Parts:
- removed C57, C58: .1uF, Capacitor_SMD:C_1206_3216Metric, symbol Xenir:Capacitor
